File: Examples/BJT_amplifier/BJT_amplifier.sch (KiCad schematic (older format))
At the start: 13 parts, among them Q1 NPN, U1 VPLOT8_1

Commit message: Change in analysis inserter GUI
Parts:
- U1: value VPLOT8_1 -> V(a)/V(b) calc
Connections:
- net labels added: a, b
Changed lines of the file:
@@
-EESchema Schematic File Version 2  date Thursday 06 June 2013 05:14:30 PM IST
+EESchema Schematic File Version 2  date Thursday 11 July 2013 03:25:19 PM IST
 LIBS:power
 LIBS:device
@@
 LIBS:contrib
 LIBS:valves
-LIBS:analogSpice
-LIBS:analogXSpice
-LIBS:convergenceAidSpice
-LIBS:converterSpice
-LIBS:digitalSpice
-LIBS:digitalXSpice
-LIBS:linearSpice
-LIBS:measurementSpice
-LIBS:portSpice
-LIBS:sourcesSpice
 LIBS:BJT_amplifier-cache
 EELAYER 25  0
@@
 Sheet 1 1
 Title ""
-Date "6 jun 2013"
+Date "11 jul 2013"
 Rev ""
 Comp ""
@@
 Comment4 ""
 $EndDescr
+Text GLabel 3750 3600 0    60   Input ~ 0
+b
+Text GLabel 5850 3900 0    60   Input ~ 0
+a
 Connection ~ 7050 4450
 Wire Wire Line
@@
 P 6800 3000
 F 0 "U1" H 6650 3100 50  0000 C CNN
-F 1 "VPLOT8_1" H 6950 3100 50  0000 C CNN
+F 1 "V(a)/V(b) calc" H 6950 3100 50  0000 C CNN
 	1    6800 3000
 	1    0    0    -1

Commit message: added vhdl and verilog
Parts:
- removed U1: V(a)/V(b) calc, symbol VPLOT8_1
- added U1: vdbplot8_1, symbol vdbplot8_1
Connections:
- net labels removed: a, b
Changed lines of the file:
@@
-EESchema Schematic File Version 2  date Thursday 11 July 2013 03:25:19 PM IST
+EESchema Schematic File Version 2  date Thursday 29 August 2013 12:29:08 PM IST
 LIBS:power
 LIBS:device
@@
 LIBS:contrib
 LIBS:valves
+LIBS:analogSpice
+LIBS:analogXSpice
+LIBS:convergenceAidSpice
+LIBS:converterSpice
+LIBS:digitalSpice
+LIBS:digitalXSpice
+LIBS:linearSpice
+LIBS:measurementSpice
+LIBS:portSpice
+LIBS:sine
+LIBS:sourcesSpice
 LIBS:BJT_amplifier-cache
 EELAYER 25  0
@@
 Sheet 1 1
 Title ""
-Date "11 jul 2013"
+Date "29 aug 2013"
 Rev ""
 Comp ""
@@
 Comment4 ""
 $EndDescr
-Text GLabel 3750 3600 0    60   Input ~ 0
-b
-Text GLabel 5850 3900 0    60   Input ~ 0
-a
+$Comp
+L vdbplot8_1 U1
+U 1 1 521AFD80
+P 6800 3000
+F 0 "U1" H 6650 3100 50  0000 C CNN
+F 1 "vdbplot8_1" H 6950 3100 50  0000 C CNN
+	1    6800 3000
+	1    0    0    -1
+$EndComp
 Connection ~ 7050 4450
 Wire Wire Line
@@
 	1    0    0    -1
 $EndComp
-$Comp
-L VPLOT8_1 U1
-U 1 1 51A5D42D
-P 6800 3000
-F 0 "U1" H 6650 3100 50  0000 C CNN
-F 1 "V(a)/V(b) calc" H 6950 3100 50  0000 C CNN
-	1    6800 3000
-	1    0    0    -1
-$EndComp
