File: Examples/sedra_smith/chapter_2/example_2.1/example_2.1.sch (KiCad schematic (older format))
At the start: 5 parts, among them U1 IPLOT

Commit message: added vhdl and verilog
Parts:
- added U2: VPLOT8, symbol VPLOT8
Connections:
- wire segments 9 -> 11
Changed lines of the file:
@@
-EESchema Schematic File Version 2  date Tuesday 14 May 2013 11:52:16 AM IST
+EESchema Schematic File Version 2  date Thursday 01 August 2013 05:17:20 PM IST
 LIBS:power
 LIBS:device
@@
 LIBS:contrib
 LIBS:valves
+LIBS:analogSpice
+LIBS:analogXSpice
+LIBS:convergenceAidSpice
+LIBS:converterSpice
+LIBS:digitalSpice
+LIBS:digitalXSpice
+LIBS:linearSpice
+LIBS:measurementSpice
+LIBS:portSpice
+LIBS:sourcesSpice
 LIBS:example_2.1-cache
 EELAYER 25  0
@@
 Sheet 1 1
 Title ""
-Date "14 may 2013"
+Date "1 aug 2013"
 Rev ""
 Comp ""
@@
 Comment4 ""
 $EndDescr
+Connection ~ 6200 3150
+Wire Wire Line
+	6200 2850 6200 3150
 Connection ~ 5750 5050
 Wire Wire Line
@@
 Wire Wire Line
 	6500 5050 5050 5050
+Wire Wire Line
+	5600 2850 5600 3150
+Connection ~ 5600 3150
+$Comp
+L VPLOT8 U2
+U 1 1 51FA4A87
+P 5900 2850
+F 0 "U2" H 5750 2950 50  0000 C CNN
+F 1 "VPLOT8" H 6050 2950 50  0000 C CNN
+	1    5900 2850
+	1    0    0    -1
+$EndComp
 $Comp
 L DC v2
